File: PCB/hackpad.kicad_pcb (KiCad board)
At the start: 2 copper layers, 76.5 x 116.5 mm, 41 parts, among them SW1 SW_Push, SW10 RotaryEncoder_Switch, SW11 SW_Push, SW12 SW_Push, SW13 SW_Push, SW14 SW_Push, SW15 SW_Push, SW16 SW_Push, SW17 SW_Push, SW2 SW_Push, SW3 SW_Push, SW4 SW_Push, SW5 SW_Push, SW6 SW_Push, SW7 SW_Push, SW8 SW_Push, SW9 SW_Push, U1 MOUDLE-SEEEDUINO-XIAO

Commit message: Rah
Routing:
- net ROW2: track 79.1 -> 78.6 mm
Changed lines of the file:
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@@
+	)
+	(segment
+		(start 126.974265 49.825735)
+		(end 127 49.8)
+		(width 0.2)
+		(layer "F.Cu")
+		(net "ROW1")
+	)
+	(segment
+		(start 115 51.000002)
+		(end 115.480737 50.519265)
+		(width 0.2)
+		(layer "F.Cu")
+		(net "ROW1")
+	)
+	(segment
+		(start 123.325735 49.825735)
+		(end 126.974265 49.825735)
+		(width 0.2)
+		(layer "F.Cu")
+		(net "ROW1")
 	)
 	(segment
@@
 	)
 	(segment
-		(start 126.258528 49.8)
-		(end 125.958528 49.5)
-		(width 0.2)
-		(layer "F.Cu")
-		(net "ROW1")
-	)
-	(segment
 		(start 141.280735 50.970735)
 		(end 137.029265 50.970735)
@@
 	)
 	(segment
+		(start 115 52.69)
+		(end 115 51.000002)
+		(width 0.2)
+		(layer "F.Cu")
+		(net "ROW1")
+	)
+	(segment
 		(start 143 52.69)
 		(end 141.280735 50.970735)
@@
 	)
 	(segment
-		(start 125.958528 49.5)
-		(end 118 49.5)
-		(width 0.2)
-		(layer "F.Cu")
-		(net "ROW1")
-	)
-	(segment
-		(start 115 51)
-		(end 115 52.69)
-		(width 0.2)
-		(layer "F.Cu")
-		(net "ROW1")
-	)
-	(segment
 		(start 115 52.69)
 		(end 112 49.69)
@@
 		(net "ROW1")
 	)
-	(segment
-		(start 115.480735 50.519265)
-		(end 115 51)
-		(width 0.2)
-		(layer "F.Cu")
-		(net "ROW1")
-	)
 	(via
 		(at 131.6 51)
@@
 	)
 	(via
+		(at 127 49.8)
+		(size 0.6)
+		(drill 0.3)
+		(layers "F.Cu" "B.Cu")
+		(net "ROW1")
+	)
+	(via
 		(at 137.029265 50.970735)
 		(size 0.6)
@@
 	)
 	(via
-		(at 118 49.5)
-		(size 0.6)
-		(drill 0.3)
-		(layers "F.Cu" "B.Cu")
-		(net "ROW1")
-	)
-	(via
-		(at 126.258528 49.8)
-		(size 0.6)
-		(drill 0.3)
-		(layers "F.Cu" "B.Cu")
-		(net "ROW1")
-	)
-	(via
-		(at 115.480735 50.519265)
+		(at 115.480737 50.519265)
+		(size 0.6)
+		(drill 0.3)
+		(layers "F.Cu" "B.Cu")
+		(net "ROW1")
+	)
+	(via
+		(at 123.325735 49.825735)
 		(size 0.6)
 		(drill 0.3)
@@
 	)
 	(segment
+		(start 129 52.5)
+		(end 129 52.69)
+		(width 0.2)
+		(layer "B.Cu")
+		(net "ROW1")
+	)
+	(segment
+		(start 115.480737 50.519265)
+		(end 122.5 50.519265)
+		(width 0.2)
+		(layer "B.Cu")
+		(net "ROW1")
+	)
+	(segment
+		(start 127 50.5)
+		(end 129 52.5)
+		(width 0.2)
+		(layer "B.Cu")
+		(net "ROW1")
+	)
+	(segment
 		(start 101 52.69)
 		(end 102.1 53.79)
@@
 	)
 	(segment
-		(start 129 52.541472)
-		(end 126.258528 49.8)
+		(start 122.5 50.519265)
+		(end 123.19353 49.825735)
 		(width 0.2)
 		(layer "B.Cu")
@@
 	)
 	(segment
-		(start 129 52.69)
-		(end 129 52.541472)
-		(width 0.2)
-		(layer "B.Cu")
-		(net "ROW1")
-	)
-	(segment
 		(start 143 49.651471)
 		(end 143 52.69)
@@
 	)
 	(segment
+		(start 127 49.8)
+		(end 127 50.5)
+		(width 0.2)
+		(layer "B.Cu")
+		(net "ROW1")
+	)
+	(segment
 		(start 113.9 53.79)
 		(end 115 52.69)
@@
 	)
 	(segment
-		(start 118 49.5)
-		(end 116.980735 50.519265)
-		(width 0.2)
-		(layer "B.Cu")
-		(net "ROW1")
-	)
-	(segment
-		(start 116.980735 50.519265)
-		(end 115.480735 50.519265)
-		(width 0.2)
-		(layer "B.Cu")
-		(net "ROW1")
-	)
-	(segment
 		(start 151.88 44)
 		(end 148.651471 44)
@@
 	)
 	(segment
+		(start 123.19353 49.825735)
+		(end 123.325735 49.825735)
+		(width 0.2)
+		(layer "B.Cu")
+		(net "ROW1")
+	)
+	(segment
 		(start 120.35 66.46)
 		(end 115 61.11)
@@
 	)
 	(segment
+		(start 127.7 49.2)
+		(end 128 49.5)
+		(width 0.2)
+		(layer "F.Cu")
+		(net "ROW2")
+	)
+	(segment
+		(start 125.025735 49.2)
+		(end 127.7 49.2)
+		(width 0.2)
+		(layer "F.Cu")
+		(net "ROW2")
+	)
+	(segment
 		(start 111.5 37.263654)
 		(end 116.463654 32.3)
@@
 	)
 	(segment
-		(start 127 48.5)
-		(end 128 49.5)
-		(width 0.2)
-		(layer "F.Cu")
-		(net "ROW2")
-	)
-	(segment
 		(start 111.5 52.69)
 		(end 111.5 37.263654)
@@
 	)
 	(segment
-		(start 125.5 48.5)
-		(end 127 48.5)
+		(start 125 49.225735)
+		(end 125.025735 49.2)
 		(width 0.2)
 		(layer "F.Cu")
@@
 	)
 	(via
+		(at 125 49.225735)
+		(size 0.6)
+		(drill 0.3)
+		(layers "F.Cu" "B.Cu")
+		(net "ROW2")
+	)
+	(via
 		(at 126.5 51)
 		(size 0.6)
@@
 	)
 	(via
-		(at 125.5 48.5)
-		(size 0.6)
-		(drill 0.3)
-		(layers "F.Cu" "B.Cu")
-		(net "ROW2")
-	)
-	(via
 		(at 128.5 51)
 		(size 0.6)
 		(drill 0.3)
 		(layers "F.Cu" "B.Cu")
-		(net "ROW2")
-	)
-	(segment
-		(start 122.880735 51.119265)
-		(end 125.5 48.5)
-		(width 0.2)
-		(layer "B.Cu")
 		(net "ROW2")
 	)
@@
 	)
 	(segment
+		(start 124.774265 49.225735)
+		(end 125 49.225735)
+		(width 0.2)
+		(layer "B.Cu")
+		(net "ROW2")
+	)
+	(segment
 		(start 112.580738 51.119265)
 		(end 122.880735 51.119265)
 		(width 0.2)
 		(layer "B.Cu")
+		(net "ROW2")
+	)
+	(segment
+		(start 122.880735 51.119265)
+		(end 124.774265 49.225735)
+		(width 0.2)
+		(layer "B.Cu")
